File: numpad/numpad.kicad_pcb (KiCad board)
At the start: 2 copper layers, 290.5 x 128.6 mm, 81 parts, among them J1 HRO_TYPE-C-31-M-12, J2 HRO_TYPE-C-31-M-12, SW1 P830, SW10 NUM2, SW11 NUM., SW12 NUM*, SW13 NUM9, SW14 NUM6, SW15 NUM3, SW16 NUM-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

Commit message: Route the rest of numpad
Parts:
- moved U2 53.3 mm to (211.9, 136.9)
- moved J1 50.5 mm to (190.3, 125.1), turned to 90 degrees
- moved C21 47.6 mm to (204.1, 121.9)
- moved C10 47.5 mm to (202.6, 120.4)
- moved C14 47.5 mm to (209.5, 126.0)
- moved C15 47.5 mm to (200.9, 125.8)
- moved C16 47.5 mm to (203.3, 132.3)
- moved C17 47.5 mm to (204.8, 132.3)
- moved C18 47.5 mm to (210.1, 122.0)
- moved C19 47.5 mm to (206.4, 132.3)
- moved C20 47.5 mm to (207.9, 132.3)
- moved C8 47.5 mm to (201.0, 120.4)
- moved FB1 47.5 mm to (199.5, 120.4)
- moved R5 47.5 mm to (200.9, 130.5)
- moved R6 47.5 mm to (200.9, 129.0)
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Connections:
- C10 pad 1: Net-(C10-Pad1) -> VBUS
- C11 pad 2: Net-(C11-Pad2) -> VBUS
- C22 pad 2: Net-(C22-Pad2) -> VBUS
- C8 pad 1: Net-(C10-Pad1) -> VBUS
- D16 pad 1: /ROW1 -> /ROW2
- D17 pad 1: /ROW3 -> /ROW4
- FB1 pad 1: Net-(C10-Pad1) -> VBUS
- FB2 pad 1: Net-(C22-Pad2) -> VBUS
- J1 pad A8: Net-(J1-PadA8) -> /ROW_FN
- J1 pad B8: Net-(J1-PadB8) -> /ROW_FN
- SW11 pad 2: /COL1 -> /COL2
- U3 pad 5: Net-(C10-Pad1) -> VBUS
- U4 pad 1: Net-(C11-Pad2) -> VBUS
- U4 pad 3: Net-(C11-Pad2) -> VBUS
- U6 pad 5: Net-(C22-Pad2) -> VBUS
Routing:
- net /ROW4: track 0.00 -> 190.7 mm
- net /ROW2: track 0.00 -> 151.0 mm, vias 0 -> 2
- net /ROW3: track 0.00 -> 144.0 mm, vias 0 -> 2
- net /COL3: track 0.00 -> 128.8 mm, vias 0 -> 1
- net /ROW0: track 0.00 -> 116.2 mm, vias 0 -> 2
- net /COL2: track 0.00 -> 112.3 mm, vias 0 -> 1
- net /ROW1: track 0.00 -> 110.5 mm
- net /COL0: track 0.00 -> 104.2 mm, vias 0 -> 1
- net /COL1: track 0.00 -> 81.1 mm, vias 0 -> 1
- net VBUS: track 0.00 -> 81.1 mm, vias 0 -> 2
- net GND: track 61.3 -> 5.50 mm, vias 22 -> 2
- net /USB_OUT_D-: track 2.30 -> 52.0 mm
- net /USB_OUT_D+: track 2.57 -> 51.8 mm
- net VUSB: track 42.9 -> 0.00 mm
- net /ROW_FN: track 31.5 -> 72.5 mm, vias 3 -> 6
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Other:
- board outline removed
- net class Power added: clearance 0.16, trace_width 0.25, via_dia 0.5, via_drill 0.3
- net class USB: trace_width 0.25 -> 0.3
