File: numpad/numpad.sch (KiCad schematic (older format))
At the start: 49 parts, among them J1 HRO_TYPE-C-31-M-12, J2 HRO_TYPE-C-31-M-12, J3 M55-7101642R, J4 M55-6101642R, SW1 P830, U1 USBLC6-2P6, U2 USBLC6-2P6, U3 MIC5504-3.3YM5, U4 STM32F042K6Ux, U5 USB2422-MJ, U6 MIC5504-3.3YM5, Y1 TSX-3225 24.0000M

Commit message: Add base numpad files
Parts:
- removed J3: M55-7101642R, eckskey:M557101642R, symbol Connector:Conn_01x16_Male
- removed J4: M55-6101642R, eckskey:M556101642R, symbol Connector:Conn_01x16_Female
- renumbered C2 to C1, C21 to C10, C5 to C11, C6 to C13, C19 to C14, C20 to C15, C13 to C16, C16 to C17, C14 to C18, C17 to C19, C22 to C2, C18 to C20, C15 to C21, C3 to C22, C4 to C23, C7 to C3, C8 to C4, C9 to C5, C23 to C6, C10 to C7, C1 to C8, C11 to C9, R3 to R1, R4 to R10, R5 to R11, R6 to R12, R1 to R2, R2 to R3, R7 to R4, R9 to R5, R10 to R6, R11 to R7, R12 to R8, R8 to R9, U6 to U1, U4 to U2, U1 to U3, U3 to U4, U2 to U6
Connections:
- wire segments 327 -> 284

Commit message: Route the rest of numpad
Connections:
- net labels added: VBUS
- net labels removed: VUSB
- wire segments 284 -> 288
- no-connect marks 11 -> 9
Changed lines of the file:
@@
 Comment4 ""
 $EndDescr
-$Comp
-L Connector:USB_C_Receptacle_USB2.0 J1
-U 1 1 5F30B828
-P 1150 1500
-F 0 "J1" H 800 2250 50  0000 C CNN
-F 1 "HRO_TYPE-C-31-M-12" H 1250 2250 31  0000 C CNN
-F 2 "Connector_USB:USB_C_Receptacle_HRO_TYPE-C-31-M-12" H 1300 1500 50  0001 C CNN
-F 3 "https://www.usb.org/sites/default/files/documents/usb_type-c.zip" H 1300 1500 50  0001 C CNN
-	1    1150 1500
-	1    0    0    -1
-$EndComp
 Entry Wire Line
 	9400 4050 9500 3950
@@
 	2500 1200 2500 1250
 $Comp
-L Copperforge:VUSB #PWR?
-U 1 1 5F8AAB27
-P 2800 850
-F 0 "#PWR?" H 2800 700 50  0001 C CNN
-F 1 "VUSB" H 2815 1023 50  0000 C CNN
-F 2 "" H 2800 850 50  0001 C CNN
-F 3 "" H 2800 850 50  0001 C CNN
-	1    2800 850
-	1    0    0    -1
-$EndComp
-$Comp
 L power:GND #PWR09
 U 1 1 5F8AB6E3
@@
 Wire Wire Line
 	3900 3750 3900 3950
-$Comp
-L Copperforge:VUSB #PWR?
-U 1 1 5F938B78
-P 2850 3450
-F 0 "#PWR?" H 2850 3300 50  0001 C CNN
-F 1 "VUSB" H 2865 3623 50  0000 C CNN
-F 2 "" H 2850 3450 50  0001 C CNN
-F 3 "" H 2850 3450 50  0001 C CNN
-	1    2850 3450
-	1    0    0    -1
-$EndComp
 $Comp
 L power:+3.3V #PWR014
@@
 Text Label 1300 5700 2    50   ~ 0
 ROW_FN
-NoConn ~ 1750 2000
-NoConn ~ 1750 2100
 Wire Wire Line
 	9950 2050 9850 2050
@@
 Wire Wire Line
 	9400 1250 9400 1300
-$Comp
-L Copperforge:VUSB #PWR?
-U 1 1 5FC66F04
-P 8950 900
-F 0 "#PWR?" H 8950 750 50  0001 C CNN
-F 1 "VUSB" H 8965 1073 50  0000 C CNN
-F 2 "" H 8950 900 50  0001 C CNN
-F 3 "" H 8950 900 50  0001 C CNN
-	1    8950 900
-	-1   0    0    -1
-$EndComp
 $Comp
 L power:GND #PWR025
@@
 Entry Wire Line
 	9400 4350 9500 4250
+$Comp
+L power:VBUS #PWR0101
+U 1 1 5F4989AA
+P 2850 3450
+F 0 "#PWR0101" H 2850 3300 50  0001 C CNN
+F 1 "VBUS" H 2865 3623 50  0000 C CNN
+F 2 "" H 2850 3450 50  0001 C CNN
+F 3 "" H 2850 3450 50  0001 C CNN
+	1    2850 3450
+	1    0    0    -1
+$EndComp
+$Comp
+L power:VBUS #PWR0102
+U 1 1 5F4A5F9A
+P 2800 850
+F 0 "#PWR0102" H 2800 700 50  0001 C CNN
+F 1 "VBUS" H 2815 1023 50  0000 C CNN
+F 2 "" H 2800 850 50  0001 C CNN
+F 3 "" H 2800 850 50  0001 C CNN
+	1    2800 850
+	1    0    0    -1
+$EndComp
+$Comp
+L power:VBUS #PWR0103
+U 1 1 5F4AF011
+P 8950 900
+F 0 "#PWR0103" H 8950 750 50  0001 C CNN
+F 1 "VBUS" H 8965 1073 50  0000 C CNN
+F 2 "" H 8950 900 50  0001 C CNN
+F 3 "" H 8950 900 50  0001 C CNN
+	1    8950 900
+	1    0    0    -1
+$EndComp
+$Comp
+L Connector:USB_C_Receptacle_USB2.0 J1
+U 1 1 5F30B828
+P 1150 1500
+F 0 "J1" H 800 2250 50  0000 C CNN
+F 1 "HRO_TYPE-C-31-M-12" H 1250 2250 31  0000 C CNN
+F 2 "Connector_USB:USB_C_Receptacle_HRO_TYPE-C-31-M-12" H 1300 1500 50  0001 C CNN
+F 3 "https://www.usb.org/sites/default/files/documents/usb_type-c.zip" H 1300 1500 50  0001 C CNN
+	1    1150 1500
+	1    0    0    -1
+$EndComp
+Wire Wire Line
+	1750 2000 1850 2000
+Wire Wire Line
+	1850 2000 1850 2100
+Wire Wire Line
+	1850 2100 1750 2100
+Wire Wire Line
+	1850 2100 1900 2100
+Connection ~ 1850 2100
+Text Label 1900 2100 0    50   ~ 0
+ROW_FN
 Wire Bus Line
 	9500 3850 9500 5250
